Commit message: Add pregrasp_handle  moveit arm configuration

File: franka_moveit_config/srdf/group_definition.xacro (robot description, xacro)
@@ -23,4 +23,13 @@
       <joint name="${arm_id}_joint7" value="${pi/4}"/>
     </group_state>
+    <group_state name="pregrasp_handle" group="${group_name}">
+      <joint name="${arm_id}_joint1" value="0.471317"/>
+      <joint name="${arm_id}_joint2" value="-0.627183"/>
+      <joint name="${arm_id}_joint3" value="-0.254263"/>
+      <joint name="${arm_id}_joint4" value="-2.062881"/>
+      <joint name="${arm_id}_joint5" value="-0.149248"/>
+      <joint name="${arm_id}_joint6" value="1.452431"/>
+      <joint name="${arm_id}_joint7" value="-0.496878"/>
+    </group_state>
   </xacro:macro>
 </robot>
